File: hardware/BatterySwitch.kicad_sch (KiCad schematic)
At the start: 63 parts, among them Q1 IRF100P219, Q2 IRF100P219, Q3 IRF100P219, Q4 IRF100P219, T1 MPSA42 (300V!), T2 MPSA42 (300V!), T3 BC547B, T4 BC547B, T5 MJE340, U1 LM393, X1 Super Soco Akku 1 (50Ah), X2 Super Soco Akku 2 (30Ah), X3 Last / Controller

Commit message: Sense-Abgriff an der Steckerklemme statt am Batteriepol dokumentiert
Bei Steckakkus (Super Soco) ist der Batteriepol nicht zugaenglich. Der
Sense-Abgriff erfolgt daher an der Anschlussklemme des Akku-Steckers im
Umschalter, vor der Hauptsicherung F1/F2 - elektrisch unkritisch:

- Abfaelle hinter dem Abgriff (F1/F2, MOSFETs) gehen nicht in die
  Messung ein (Sense-Zweig zieht nur ~1 mA)
- Der Abfall ueber Akkukabel/Steckerkontakt (~0,1-0,3 V bei 40 A)
  wirkt nur beim aktiven Akku, in dieselbe Richtung wie der Last-
  einbruch, und wird beim Einstellen von Delta mit beruecksichtigt
- Voraussetzung: beide Akkuzuleitungen gleich ausfuehren
  (Querschnitt, Laenge, Steckertyp)

Formulierungen in Schaltungsbeschreibung, Aufbauanleitung, README,
Stueckliste und im Schaltplan-Hinweistext angepasst.

Co-Authored-By: Claude Fable 5 <noreply@anthropic.com>
Claude-Session: https://claude.ai/code/session_011gicRxuedseUphnQpmYx5w
Other:
- note added: "Sense-Abgriff direkt an der Akku-Steckerklemme (vor F1/F2)!"
- note removed: "Sense-Leitungen direkt am Batteriepol abgreifen!"
